File: hw/subtractMod/In_channel.kicad_sch (KiCad schematic)
At the start: 21 parts, among them IC1 AD8244, J1 Screw_Terminal_01x04, J2 Screw_Terminal_01x04, U3 AD8276, U4 AD8276

Commit message: updated schematics of subtraction module
Parts:
- RV1: renamed from RV5; footprint (none) -> Potentiometer_SMD:Potentiometer_Bourns_3314J_Vertical
- RV2: renamed from RV6; footprint (none) -> Potentiometer_SMD:Potentiometer_Bourns_3314J_Vertical
- renumbered C3 to C1, C4 to C2, J2 to J1, J1 to J2, R6 to R1, R7 to R2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
