File: hw/subtractMod/offset_ctrl.kicad_sch (KiCad schematic)
At the start: 9 parts, among them IC2 LMP2011, U2 AD8276

Commit message: updated schematics of subtraction module
Parts:
- RV3: renamed from RV1; footprint (none) -> Potentiometer_SMD:Potentiometer_Bourns_3314J_Vertical
- RV4: renamed from RV2; footprint (none) -> Potentiometer_SMD:Potentiometer_Bourns_3314J_Vertical
- RV5: renamed from RV3; footprint (none) -> Potentiometer_SMD:Potentiometer_Bourns_3314J_Vertical
- RV6: renamed from RV4; footprint (none) -> Potentiometer_SMD:Potentiometer_Bourns_3314J_Vertical
- renumbered TP6 to TP10, TP13 to TP11, U2 to U4
Changed lines of the file:
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@@
 		(on_board yes)
 		(dnp no)
-		(property "Reference" "U2"
+		(property "Reference" "U4"
 			(at 171.45 106.68 0)
 			(effects
@@
 		(pin "8"
 		)
+		(instances
+			(project ""
+				(path "/900e6e10-af1f-4ec5-a075-6ae6c64aeb78/00000000-0000-0000-0000-00005e556d6f"
+					(reference "U4")
+					(unit 1)
+				)
+			)
+		)
 	)
 	(symbol
@@
 		(on_board yes)
 		(dnp no)
-		(property "Reference" "#PWR07"
+		(property "Reference" "#PWR023"
 			(at 163.83 115.57 0)
 			(effects
@@
 		(pin "1"
 		)
+		(instances
+			(project ""
+				(path "/900e6e10-af1f-4ec5-a075-6ae6c64aeb78/00000000-0000-0000-0000-00005e556d6f"
+					(reference "#PWR023")
+					(unit 1)
+				)
+			)
+		)
 	)
 	(symbol
@@
 		(on_board yes)
 		(dnp no)
-		(property "Reference" "#PWR06"
+		(property "Reference" "#PWR022"
 			(at 163.83 93.98 0)
 			(effects
@@
 		(pin "1"
 		)
+		(instances
+			(project ""
+				(path "/900e6e10-af1f-4ec5-a075-6ae6c64aeb78/00000000-0000-0000-0000-00005e556d6f"
+					(reference "#PWR022")
+					(unit 1)
+				)
+			)
+		)
 	)
 	(symbol
@@
 		(on_board yes)
 		(dnp no)
-		(property "Reference" "#PWR08"
+		(property "Reference" "#PWR024"
 			(at 171.45 118.11 0)
 			(effects
@@
 		(pin "1"
 		)
+		(instances
+			(project ""
+				(path "/900e6e10-af1f-4ec5-a075-6ae6c64aeb78/00000000-0000-0000-0000-00005e556d6f"
+					(reference "#PWR024")
+					(unit 1)
+				)
+			)
+		)
 	)
 	(symbol
@@
 		(on_board yes)
 		(dnp no)
-		(property "Reference" "#PWR09"
+		(property "Reference" "#PWR026"
 			(at 226.06 66.04 0)
 			(effects
@@
 		(pin "1"
 		)
+		(instances
+			(project ""
+				(path "/900e6e10-af1f-4ec5-a075-6ae6c64aeb78/00000000-0000-0000-0000-00005e556d6f"
+					(reference "#PWR026")
+					(unit 1)
+				)
+			)
+		)
 	)
 	(symbol
@@
 		(on_board yes)
 		(dnp no)
-		(property "Reference" "#PWR010"
+		(property "Reference" "#PWR027"
 			(at 226.06 87.63 0)
 			(effects
@@
 		(pin "1"
 		)
+		(instances
+			(project ""
+				(path "/900e6e10-af1f-4ec5-a075-6ae6c64aeb78/00000000-0000-0000-0000-00005e556d6f"
+					(reference "#PWR027")
+					(unit 1)
+				)
+			)
+		)
 	)
 	(symbol
@@
 		(on_board yes)
 		(dnp no)
-		(property "Reference" "#PWR05"
+		(property "Reference" "#PWR021"
 			(at 147.32 110.49 0)
 			(effects
@@
 		(pin "1"
 		)
+		(instances
+			(project ""
+				(path "/900e6e10-af1f-4ec5-a075-6ae6c64aeb78/00000000-0000-0000-0000-00005e556d6f"
+					(reference "#PWR021")
+					(unit 1)
+				)
+			)
+		)
 	)
 	(symbol
@@
 		(on_board yes)
 		(dnp no)
-		(property "Reference" "#PWR04"
+		(property "Reference" "#PWR020"
 			(at 135.89 119.38 0)
 			(effects
@@
 		(pin "1"
 		)
+		(instances
+			(project ""
+				(path "/900e6e10-af1f-4ec5-a075-6ae6c64aeb78/00000000-0000-0000-0000-00005e556d6f"
+					(reference "#PWR020")
+					(unit 1)
+				)
+			)
+		)
 	)
 	(symbol
@@
 		(on_board yes)
 		(dnp no)
-		(property "Reference" "TP6"
+		(property "Reference" "TP10"
 			(at 182.5752 94.0816 90)
 			(effects
@@
 		(pin "1"
 		)
+		(instances
+			(project ""
+				(path "/900e6e10-af1f-4ec5-a075-6ae6c64aeb78/00000000-0000-0000-0000-00005e556d6f"
+					(reference "TP10")
+					(unit 1)
+				)
+			)
+		)
 	)
 	(symbol
@@
 		(on_board yes)
 		(dnp no)
-		(property "Reference" "#PWR027"
+		(property "Reference" "#PWR025"
 			(at 212.09 119.38 0)
 			(effects
@@
 			(project ""
 				(path "/900e6e10-af1f-4ec5-a075-6ae6c64aeb78/00000000-0000-0000-0000-00005e556d6f"
-					(reference "#PWR027")
+					(reference "#PWR025")
 					(unit 1)
 				)
@@
 		(on_board yes)
 		(dnp no)
-		(property "Reference" "TP13"
+		(property "Reference" "TP11"
 			(at 223.2152 100.4316 90)
 			(effects
@@
 			(project ""
 				(path "/900e6e10-af1f-4ec5-a075-6ae6c64aeb78/00000000-0000-0000-0000-00005e556d6f"
-					(reference "TP13")
+					(reference "TP11")
 					(unit 1)
 				)
@@
 		(dnp no)
 		(fields_autoplaced yes)
-		(property "Reference" "RV4"
+		(property "Reference" "RV6"
 			(at 200.66 105.41 90)
 			(effects
@@
 			)
 		)
-		(property "Footprint" ""
+		(property "Footprint" "Potentiometer_SMD:Potentiometer_Bourns_3314J_Vertical"
 			(at 200.66 101.6 0)
 			(effects
@@
 			(project "subtractMod"
 				(path "/900e6e10-af1f-4ec5-a075-6ae6c64aeb78/00000000-0000-0000-0000-00005e556d6f"
-					(reference "RV4")
+					(reference "RV6")
 					(unit 1)
 				)
@@
 		(dnp no)
 		(fields_autoplaced yes)
-		(property "Reference" "RV1"
+		(property "Reference" "RV3"
 			(at 129.54 82.55 90)
 			(effects
@@
 			)
 		)
-		(property "Footprint" ""
+		(property "Footprint" "Potentiometer_SMD:Potentiometer_Bourns_3314J_Vertical"
 			(at 129.54 88.9 0)
 			(effects
@@
 			(project ""
 				(path "/900e6e10-af1f-4ec5-a075-6ae6c64aeb78/00000000-0000-0000-0000-00005e556d6f"
-					(reference "RV1")
+					(reference "RV3")
 					(unit 1)
 				)
@@
 		(dnp no)
 		(fields_autoplaced yes)
-		(property "Reference" "RV2"
+		(property "Reference" "RV4"
 			(at 129.54 111.76 90)
 			(effects
@@
 			)
 		)
-		(property "Footprint" ""
+		(property "Footprint" "Potentiometer_SMD:Potentiometer_Bourns_3314J_Vertical"
 			(at 129.54 107.95 0)
 			(effects
@@
 			(project "subtractMod"
 				(path "/900e6e10-af1f-4ec5-a075-6ae6c64aeb78/00000000-0000-0000-0000-00005e556d6f"
-					(reference "RV2")
+					(reference "RV4")
 					(unit 1)
 				)
@@
 		(dnp no)
 		(fields_autoplaced yes)
-		(property "Reference" "RV3"
+		(property "Reference" "RV5"
 			(at 153.67 114.3 90)
 			(effects
@@
 			)
 		)
-		(property "Footprint" ""
+		(property "Footprint" "Potentiometer_SMD:Potentiometer_Bourns_3314J_Vertical"
 			(at 153.67 110.49 0)
 			(effects
@@
 			(project "subtractMod"
 				(path "/900e6e10-af1f-4ec5-a075-6ae6c64aeb78/00000000-0000-0000-0000-00005e556d6f"
-					(reference "RV3")
-					(unit 1)
-				)
+					(reference "RV5")
+					(unit 1)
+				)
