File: hw/subtractMod/power_block.kicad_sch (KiCad schematic)
At the start: 9 parts, among them J3 Screw_Terminal_01x02, U1 TLV6001DCK

Commit message: updated schematics of subtraction module
Parts:
- C3: renamed from C2; footprint (none) -> Capacitor_SMD:CP_Elec_6.3x5.9
- C4: renamed from C1; footprint (none) -> Capacitor_SMD:CP_Elec_6.3x5.9
- renumbered R1 to R6, R2 to R7, TP3 to TP7, TP4 to TP8, TP5 to TP9, U1 to U3
Changed lines of the file:
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@@
 		(on_board yes)
 		(dnp no)
-		(property "Reference" "R1"
+		(property "Reference" "R6"
 			(at 124.968 77.5716 0)
 			(effects
@@
 		(pin "1"
 		)
+		(instances
+			(project ""
+				(path "/900e6e10-af1f-4ec5-a075-6ae6c64aeb78/00000000-0000-0000-0000-00005e46b34f"
+					(reference "R6")
+					(unit 1)
+				)
+			)
+		)
 	)
 	(symbol
@@
 		(on_board yes)
 		(dnp no)
-		(property "Reference" "R2"
+		(property "Reference" "R7"
 			(at 124.968 100.4316 0)
 			(effects
@@
 		(pin "1"
 		)
+		(instances
+			(project ""
+				(path "/900e6e10-af1f-4ec5-a075-6ae6c64aeb78/00000000-0000-0000-0000-00005e46b34f"
+					(reference "R7")
+					(unit 1)
+				)
+			)
+		)
 	)
 	(symbol
@@
 		(on_board yes)
 		(dnp no)
-		(property "Reference" "U1"
+		(property "Reference" "U3"
 			(at 156.0576 87.7316 0)
 			(effects
@@
 		(pin "4"
 		)
+		(instances
+			(project ""
+				(path "/900e6e10-af1f-4ec5-a075-6ae6c64aeb78/00000000-0000-0000-0000-00005e46b34f"
+					(reference "U3")
+					(unit 1)
+				)
+			)
+		)
 	)
 	(symbol
@@
 		(on_board yes)
 		(dnp no)
-		(property "Reference" "TP3"
+		(property "Reference" "TP7"
 			(at 183.8452 71.2216 90)
 			(effects
@@
 		(pin "1"
 		)
+		(instances
+			(project ""
+				(path "/900e6e10-af1f-4ec5-a075-6ae6c64aeb78/00000000-0000-0000-0000-00005e46b34f"
+					(reference "TP7")
+					(unit 1)
+				)
+			)
+		)
 	)
 	(symbol
@@
 		(on_board yes)
 		(dnp no)
-		(property "Reference" "TP5"
+		(property "Reference" "TP9"
 			(at 183.8452 109.3216 90)
 			(effects
@@
 		(pin "1"
 		)
+		(instances
+			(project ""
+				(path "/900e6e10-af1f-4ec5-a075-6ae6c64aeb78/00000000-0000-0000-0000-00005e46b34f"
+					(reference "TP9")
+					(unit 1)
+				)
+			)
+		)
 	)
 	(symbol
@@
 		(on_board yes)
 		(dnp no)
-		(property "Reference" "#PWR03"
+		(property "Reference" "#PWR019"
 			(at 177.8 107.95 0)
 			(effects
@@
 		(pin "1"
 		)
+		(instances
+			(project ""
+				(path "/900e6e10-af1f-4ec5-a075-6ae6c64aeb78/00000000-0000-0000-0000-00005e46b34f"
+					(reference "#PWR019")
+					(unit 1)
+				)
+			)
+		)
 	)
 	(symbol
@@
 		(pin "1"
 		)
+		(instances
+			(project ""
+				(path "/900e6e10-af1f-4ec5-a075-6ae6c64aeb78/00000000-0000-0000-0000-00005e46b34f"
+					(reference "J3")
+					(unit 1)
+				)
+			)
+		)
 	)
 	(symbol
@@
 		(on_board yes)
 		(dnp no)
-		(property "Reference" "#PWR02"
+		(property "Reference" "#PWR018"
 			(at 177.8 76.2 0)
 			(effects
@@
 		(pin "1"
 		)
+		(instances
+			(project ""
+				(path "/900e6e10-af1f-4ec5-a075-6ae6c64aeb78/00000000-0000-0000-0000-00005e46b34f"
+					(reference "#PWR018")
+					(unit 1)
+				)
+			)
+		)
 	)
 	(symbol
@@
 		(on_board yes)
 		(dnp no)
-		(property "Reference" "TP4"
+		(property "Reference" "TP8"
 			(at 183.8452 87.7316 90)
 			(effects
@@
 		(pin "1"
 		)
+		(instances
+			(project ""
+				(path "/900e6e10-af1f-4ec5-a075-6ae6c64aeb78/00000000-0000-0000-0000-00005e46b34f"
+					(reference "TP8")
+					(unit 1)
+				)
+			)
+		)
 	)
 	(symbol
@@
 		(on_board yes)
 		(dnp no)
-		(property "Reference" "#PWR01"
+		(property "Reference" "#PWR017"
 			(at 158.75 106.68 0)
 			(effects
@@
 		(pin "1"
 		)
+		(instances
+			(project ""
+				(path "/900e6e10-af1f-4ec5-a075-6ae6c64aeb78/00000000-0000-0000-0000-00005e46b34f"
+					(reference "#PWR017")
+					(unit 1)
+				)
+			)
+		)
 	)
 	(symbol
@@
 		(dnp no)
 		(fields_autoplaced yes)
-		(property "Reference" "C1"
+		(property "Reference" "C4"
 			(at 176.53 99.4409 0)
 			(effects
@@
 			)
 		)
-		(property "Footprint" ""
+		(property "Footprint" "Capacitor_SMD:CP_Elec_6.3x5.9"
 			(at 173.6852 105.41 0)
 			(effects
@@
 			(project ""
 				(path "/900e6e10-af1f-4ec5-a075-6ae6c64aeb78/00000000-0000-0000-0000-00005e46b34f"
-					(reference "C1")
+					(reference "C4")
 					(unit 1)
 				)
@@
 		(dnp no)
 		(fields_autoplaced yes)
-		(property "Reference" "C2"
+		(property "Reference" "C3"
 			(at 176.53 77.8509 0)
 			(effects
@@
 			)
 		)
-		(property "Footprint" ""
+		(property "Footprint" "Capacitor_SMD:CP_Elec_6.3x5.9"
 			(at 173.6852 83.82 0)
 			(effects
@@
 			(project "subtractMod"
 				(path "/900e6e10-af1f-4ec5-a075-6ae6c64aeb78/00000000-0000-0000-0000-00005e46b34f"
-					(reference "C2")
-					(unit 1)
-				)
+					(reference "C3")
+					(unit 1)
+				)
