File: hw/load_cell_amplifier/load_cell_amplifier.kicad_sch (KiCad schematic)
At the start: 15 parts, among them SW1 SW_DPST_x2, U1 INA129, U2 TL072, U3 TL072

Commit message: updated kicad version
Other:
- note removed: "A = ???"
Changed lines of the file:
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@@
 (kicad_sch
-	(version 20250222)
+	(version 20250318)
 	(generator "eeschema")
 	(generator_version "9.99")
@@
 		(exclude_from_sim no)
 		(at 141.224 28.702 0)
-		(effects
-			(font
-				(size 1.27 1.27)
-			)
-		)
-	)
-	(text "A = ???"
-		(exclude_from_sim no)
-		(at 119.38 92.964 0)
 		(effects
 			(font
@@
 			)
 		)
-		(property "Datasheet" "~"
+		(property "Datasheet" ""
 			(at 207.01 110.49 0)
 			(hide yes)
@@
 			)
 		)
-		(property "Datasheet" "~"
+		(property "Datasheet" ""
 			(at 91.44 92.71 0)
 			(hide yes)
@@
 			)
 		)
-		(property "Datasheet" "~"
+		(property "Datasheet" ""
 			(at 144.78 127 0)
 			(hide yes)
@@
 			)
 		)
-		(property "Datasheet" "~"
+		(property "Datasheet" ""
 			(at 161.29 116.84 0)
 			(hide yes)
@@
 			)
 		)
-		(property "Datasheet" "~"
+		(property "Datasheet" ""
 			(at 55.88 49.53 0)
 			(hide yes)
@@
 			)
 		)
-		(property "Datasheet" "~"
+		(property "Datasheet" ""
 			(at 106.68 92.71 0)
 			(hide yes)
@@
 			)
 		)
-		(property "Datasheet" "~"
+		(property "Datasheet" ""
 			(at 223.52 102.87 0)
 			(hide yes)
@@
 			)
 		)
-		(property "Datasheet" "~"
+		(property "Datasheet" ""
 			(at 55.88 39.37 0)
 			(hide yes)
@@
 			)
 		)
-		(property "Datasheet" "~"
+		(property "Datasheet" ""
 			(at 198.12 128.27 0)
 			(hide yes)
@@
 			)
 		)
-		(property "Datasheet" "~"
+		(property "Datasheet" ""
 			(at 161.29 102.87 0)
 			(hide yes)
@@
 			)
 		)
-		(property "Datasheet" "~"
+		(property "Datasheet" ""
 			(at 207.01 119.38 0)
 			(hide yes)
@@
 			)
 		)
-		(property "Datasheet" "~"
+		(property "Datasheet" ""
 			(at 91.44 82.55 0)
 			(hide yes)
